File: 02_pcb/mouse_codename/double_ldo_design.brd (EAGLE design)
At the start: 45 x 50 mm, 8 parts, among them IC1 STM32F405RGT6, IC2 MPU-6050, IC3 DRV88361

Commit message: pcb design updated
Parts:
- added C1, C10, C2, C6, C8, C9: 100n, rcl:C0402
- added C3, C4: 2.2u, rcl:C0402
- added C5: 4.7u, rcl:C0402
- added C7: 1u, rcl:C0402
- added R1: 47k, rcl:R0402
- added R2: 10k, rcl:R0402
- added S4: B3U-3000PB3U-3000P, parts:B3U-3000P
Connections:
- new net N$1: R2.2, S3.2
- new net N$2: IC1.60, R1.2, S3.1
Changed lines of the file:
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@@
 <drawing>
 <settings>
-<setting alwaysvectorfont="yes"/>
+<setting alwaysvectorfont="no"/>
 <setting verticaltext="up"/>
 </settings>
@@
 <attribute name="VALUE" x="42.478903125" y="1.647490625" size="1.27" layer="27" rot="R45" align="center"/>
 </element>
+<element name="C1" library="rcl" library_urn="urn:adsk.eagle:library:334" package="C0402" package3d_urn="urn:adsk.eagle:package:23626/2" value="100n" x="0" y="-8.89" smashed="yes">
+<attribute name="NAME" x="-0.635" y="-8.255" size="1.27" layer="25"/>
+<attribute name="SPICEPREFIX" value="C" x="0" y="-8.89" size="1.778" layer="27" display="off"/>
+<attribute name="VALUE" x="-0.635" y="-10.795" size="1.27" layer="27"/>
+</element>
+<element name="C2" library="rcl" library_urn="urn:adsk.eagle:library:334" package="C0402" package3d_urn="urn:adsk.eagle:package:23626/2" value="100n" x="0" y="-13.97" smashed="yes">
+<attribute name="NAME" x="-0.635" y="-13.335" size="1.27" layer="25"/>
+<attribute name="SPICEPREFIX" value="C" x="0" y="-13.97" size="1.778" layer="27" display="off"/>
+<attribute name="VALUE" x="-0.635" y="-15.875" size="1.27" layer="27"/>
+</element>
+<element name="C3" library="rcl" library_urn="urn:adsk.eagle:library:334" package="C0402" package3d_urn="urn:adsk.eagle:package:23626/2" value="2.2u" x="0" y="-19.05" smashed="yes">
+<attribute name="NAME" x="-0.635" y="-18.415" size="1.27" layer="25"/>
+<attribute name="SPICEPREFIX" value="C" x="0" y="-19.05" size="1.778" layer="27" display="off"/>
+<attribute name="VALUE" x="-0.635" y="-20.955" size="1.27" layer="27"/>
+</element>
+<element name="C4" library="rcl" library_urn="urn:adsk.eagle:library:334" package="C0402" package3d_urn="urn:adsk.eagle:package:23626/2" value="2.2u" x="0" y="-24.13" smashed="yes">
+<attribute name="NAME" x="-0.635" y="-23.495" size="1.27" layer="25"/>
+<attribute name="SPICEPREFIX" value="C" x="0" y="-24.13" size="1.778" layer="27" display="off"/>
+<attribute name="VALUE" x="-0.635" y="-26.035" size="1.27" layer="27"/>
+</element>
+<element name="C5" library="rcl" library_urn="urn:adsk.eagle:library:334" package="C0402" package3d_urn="urn:adsk.eagle:package:23626/2" value="4.7u" x="0" y="-29.21" smashed="yes">
+<attribute name="NAME" x="-0.635" y="-28.575" size="1.27" layer="25"/>
+<attribute name="SPICEPREFIX" value="C" x="0" y="-29.21" size="1.778" layer="27" display="off"/>
+<attribute name="VALUE" x="-0.635" y="-31.115" size="1.27" layer="27"/>
+</element>
+<element name="C6" library="rcl" library_urn="urn:adsk.eagle:library:334" package="C0402" package3d_urn="urn:adsk.eagle:package:23626/2" value="100n" x="0" y="-34.29" smashed="yes">
+<attribute name="NAME" x="-0.635" y="-33.655" size="1.27" layer="25"/>
+<attribute name="SPICEPREFIX" value="C" x="0" y="-34.29" size="1.778" layer="27" display="off"/>
+<attribute name="VALUE" x="-0.635" y="-36.195" size="1.27" layer="27"/>
+</element>
+<element name="C7" library="rcl" library_urn="urn:adsk.eagle:library:334" package="C0402" package3d_urn="urn:adsk.eagle:package:23626/2" value="1u" x="0" y="-39.37" smashed="yes">
+<attribute name="NAME" x="-0.635" y="-38.735" size="1.27" layer="25"/>
+<attribute name="SPICEPREFIX" value="C" x="0" y="-39.37" size="1.778" layer="27" display="off"/>
+<attribute name="VALUE" x="-0.635" y="-41.275" size="1.27" layer="27"/>
+</element>
+<element name="R1" library="rcl" library_urn="urn:adsk.eagle:library:334" package="R0402" package3d_urn="urn:adsk.eagle:package:23547/3" value="47k" x="0" y="-44.45" smashed="yes">
+<attribute name="NAME" x="-0.635" y="-43.815" size="1.27" layer="25"/>
+<attribute name="SPICEPREFIX" value="R" x="0" y="-44.45" size="1.778" layer="27" display="off"/>
+<attribute name="VALUE" x="-0.635" y="-46.355" size="1.27" layer="27"/>
+</element>
+<element name="R2" library="rcl" library_urn="urn:adsk.eagle:library:334" package="R0402" package3d_urn="urn:adsk.eagle:package:23547/3" value="10k" x="0" y="-48.26" smashed="yes">
+<attribute name="NAME" x="-0.635" y="-47.625" size="1.27" layer="25"/>
+<attribute name="SPICEPREFIX" value="R" x="0" y="-48.26" size="1.778" layer="27" display="off"/>
+<attribute name="VALUE" x="-0.635" y="-50.165" size="1.27" layer="27"/>
+</element>
+<element name="S4" library="parts" library_urn="urn:adsk.eagle:library:8879268" package="B3U-3000P" package3d_urn="urn:adsk.eagle:package:8879469/3" value="B3U-3000PB3U-3000P" x="3.81" y="-54.61" smashed="yes">
+<attribute name="NAME" x="3.349" y="-52.403" size="1.27" layer="25" align="center"/>
+<attribute name="VALUE" x="3.222" y="-56.721" size="1.27" layer="27" align="center"/>
+</element>
+<element name="C8" library="rcl" library_urn="urn:adsk.eagle:library:334" package="C0402" package3d_urn="urn:adsk.eagle:package:23626/2" value="100n" x="-5.08" y="-60.96" smashed="yes">
+<attribute name="NAME" x="-5.715" y="-60.325" size="1.27" layer="25"/>
+<attribute name="SPICEPREFIX" value="C" x="-5.08" y="-60.96" size="1.778" layer="27" display="off"/>
+<attribute name="VALUE" x="-5.715" y="-62.865" size="1.27" layer="27"/>
+</element>
+<element name="C9" library="rcl" library_urn="urn:adsk.eagle:library:334" package="C0402" package3d_urn="urn:adsk.eagle:package:23626/2" value="100n" x="-5.08" y="-66.04" smashed="yes">
+<attribute name="NAME" x="-5.715" y="-65.405" size="1.27" layer="25"/>
+<attribute name="SPICEPREFIX" value="C" x="-5.08" y="-66.04" size="1.778" layer="27" display="off"/>
+<attribute name="VALUE" x="-5.715" y="-67.945" size="1.27" layer="27"/>
+</element>
+<element name="C10" library="rcl" library_urn="urn:adsk.eagle:library:334" package="C0402" package3d_urn="urn:adsk.eagle:package:23626/2" value="100n" x="-5.08" y="-71.12" smashed="yes">
+<attribute name="NAME" x="-5.715" y="-70.485" size="1.27" layer="25"/>
+<attribute name="SPICEPREFIX" value="C" x="-5.08" y="-71.12" size="1.778" layer="27" display="off"/>
+<attribute name="VALUE" x="-5.715" y="-73.025" size="1.27" layer="27"/>
+</element>
 </elements>
 <signals>
@@
 <contactref element="IC1" pad="63"/>
 </signal>
+<signal name="N$1">
+<contactref element="R2" pad="2"/>
+<contactref element="S3" pad="2"/>
+<wire x1="40.199915625" y1="2.353915625" x2="0.5" y2="-48.26" width="0" layer="19" extent="1-1"/>
+</signal>
+<signal name="N$2">
+<contactref element="S3" pad="1"/>
+<contactref element="IC1" pad="60"/>
+<contactref element="R1" pad="2"/>
+<wire x1="42.60408125" y1="4.75808125" x2="21.11" y2="38.77" width="0" layer="19" extent="1-1"/>
+<wire x1="0.5" y1="-44.45" x2="42.60408125" y2="4.75808125" width="0" layer="19" extent="1-1"/>
+</signal>
 </signals>

Commit message: pcb updated
Parts:
- added C11, C12, C13: 100n, rcl:C0402
- added R3: 10k, rcl:R0402
- C3, C4: value 2.2u -> 100n
- C8, C9: value 100n -> 2.2u
- IC1: value STM32F405RGT6 -> STM32F405RGT6_L
- R1: value 47k -> 1k
- S2, S3: value B3U-3000PB3U-3000P -> B3U-3000P
- S4: value B3U-3000PB3U-3000P -> B3U-1000P; device parts:B3U-3000P -> parts:B3U-1000P
- moved C10 110.7 mm to (-11.4, 39.4)
- moved S4 90.9 mm to (-7.62, 35.6)
- moved C3 69.5 mm to (-11.4, 49.5)
- moved C4 69.5 mm to (-11.4, 44.5)
- moved C9 61.4 mm to (2.54, -5.08), flipped to the bottom, turned to 270 degrees
- moved R1 58.3 mm to (-11.4, 12.7)
- moved R2 58.3 mm to (-11.4, 8.89)
- moved C8 57.3 mm to (7.62, -5.08), flipped to the bottom, turned to 270 degrees
- moved S3 51.4 mm to (-7.62, 19.1), turned to 0 degrees
- moved C7 36.6 mm to (-12.7, -5.08), flipped to the bottom, turned to 270 degrees
- moved C6 30.2 mm to (-7.62, -5.08), flipped to the bottom, turned to 270 degrees
- moved S2 29.5 mm to (-7.62, 26.7)
- moved S1 29.2 mm to (-7.62, 31.8)
- moved C5 24.3 mm to (-2.54, -5.08), flipped to the bottom, turned to 270 degrees
- moved C1 18.2 mm to (17.8, -5.08), flipped to the bottom, turned to 270 degrees
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Connections:
- removed net N$1: R2.2, S3.2
- removed net VDDA: IC1.13
- removed net VDD_1: IC1.19
- removed net VDD_2: IC1.32
- removed net VDD_3: IC1.48
- removed net VDD_4: IC1.64
- removed net VSSA: IC1.12
- removed net VSS_1: IC1.18
- removed net VSS_2: IC1.63
- new net +3V3: C1.1, C10.1, C2.1, C3.1, C4.1, C5.1, C6.1, C7.1, C8.1, C9.1, IC1.13, IC1.19, IC1.31, IC1.32, IC1.47, IC1.48, IC1.64, R1.2
- new net BOOT0: IC1.60, R3.2, S3.1
- new net BOOT1: IC1.28, R2.2
- new net BTN1: C12.1, IC1.50, S2.2
- new net BTN2: C13.1, IC1.49, S4.2
- new net ENC1_CHA: IC1.41
- new net ENC1_CHB: IC1.42
- new net GND: C1.2, C11.2, C12.2, C13.2, C2.2, C3.2, C4.2, C5.2, C6.2, C7.2, C8.2, C9.2, IC1.12, IC1.18, IC1.63, R2.1, R3.1, S1.1, S2.1, S4.1
- new net IRD1: IC1.16
- new net IRD2: IC1.17
- new net N$10: C10.2, IC1.1
- new net NRST: C11.1, IC1.7, S1.2
- new net PTR1: IC1.14
- new net PTR2: IC1.15
- net N$2: now also R1.1, S3.2; no longer IC1.60, R1.2, S3.1
