File: 02_pcb/mouse_codename/double_ldo_design.sch (EAGLE design)
At the start: 21 parts, among them IC1 STM32F405RGT6, IC2 MPU-6050, IC3 DRV88361

Commit message: pcb updated
Parts:
- added C11, C12, C13: 100n, rcl:C-USC0402
- added R3: 10k, rcl:R-US_R0402
- C3, C4: value 2.2u -> 100n
- C8, C9: value 100n -> 2.2u
- IC1: value STM32F405RGT6 -> STM32F405RGT6_L; device parts:STM32F405RGT6 -> parts:STM32F405RGT6_L
- R1: value 47k -> 1k
- S2, S3: value B3U-3000PB3U-3000P -> B3U-3000P; device parts:B3U-3000PB3U-3000P -> parts:B3U-3000P
- S4: value B3U-3000PB3U-3000P -> B3U-1000P; device parts:B3U-3000PB3U-3000P -> parts:B3U-1000P
Connections:
- removed net N$1: R2.2, S3.2
- new net +3V3: C1.1, C10.1, C2.1, C3.1, C4.1, C5.1, C6.1, C7.1, C8.1, C9.1, IC1.VCAP_1, IC1.VCAP_2, IC1.VDDA, IC1.VDD_1, IC1.VDD_2, IC1.VDD_3, IC1.VDD_4, R1.2
- new net BOOT0: IC1.BOOT0, R3.2, S3.1
- new net BOOT1: IC1.PB2/BOOT1, R2.2
- new net BTN1: C12.1, IC1.PA15, S2.2
- new net BTN2: C13.1, IC1.PA14, S4.2
- new net ENC1_CHA: IC1.PA8
- new net ENC1_CHB: IC1.PA9
- new net GND: C1.2, C11.2, C12.2, C13.2, C2.2, C3.2, C4.2, C5.2, C6.2, C7.2, C8.2, C9.2, IC1.VSSA, IC1.VSS_1, IC1.VSS_2, R2.1, R3.1, S1.1, S2.1, S4.1
- new net IRD1: IC1.PA2
- new net IRD2: IC1.PA3
- new net N$10: C10.2, IC1.VBAT
- new net NRST: C11.1, IC1.NRST, S1.2
- new net PTR1: IC1.PA0_WKUP
- new net PTR2: IC1.PA1
- net N$2: now also R1.1, S3.2; no longer IC1.BOOT0, R1.2, S3.1
Other:
- note added: "The V BAT pin can be connected to the external battery (1.65 V < V BAT < 3.6 V). If no external battery is used, it is recommended to connect this pin to V DD with a 100 nF external ceramic decoupling capacitor."
- moved on the sheet: C1, C10, C2, C3, C4, C5, C6, C7, C8, C9, IC1, R1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
