File: 02_pcb/mouse_codename/micromouse2019_enc.sch (EAGLE design)
At the start: 7 parts, among them IC1 AS5047D

Commit message: Enc pcb updated, design rules trace to dim updated
Parts:
- removed U$1: CONN_SPI, 0-micromouse2019:CONN_SPI
- added CONN1: CONN_SPI-P127, 0-micromouse2019:CONN_SPI-P127
- PORT1: value ENC_PORT_MODULE -> PORT_ENC_MODULE; device 0-micromouse2019:ENC_PORT_MODULE -> 0-micromouse2019:PORT_ENC_MODULE
Connections:
- net CLK: now also CONN1.P2; no longer U$1.P3
- net CSN: now also CONN1.P1; no longer U$1.P4
- net MISO: now also CONN1.P3; no longer U$1.P2
- net MOSI: now also CONN1.P4; no longer U$1.P1
Changed lines of the file:
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@@
 <part name="GND6" library="0-micromouse2019" deviceset="GND" device=""/>
 <part name="+3V3" library="0-micromouse2019" deviceset="+3V3" device=""/>
-<part name="PORT1" library="0-micromouse2019" deviceset="ENC_PORT" device="_MODULE"/>
+<part name="PORT1" library="0-micromouse2019" deviceset="PORT_ENC" device="_MODULE"/>
 <part name="FRAME1" library="frames" library_urn="urn:adsk.eagle:library:229" deviceset="DINA4_L" device=""/>
-<part name="U$1" library="0-micromouse2019" deviceset="CONN_SPI" device="" package3d_urn="urn:adsk.eagle:package:9165666/2"/>
+<part name="CONN1" library="0-micromouse2019" deviceset="CONN_SPI" device="-P127" package3d_urn="urn:adsk.eagle:package:9165666/2"/>
 </parts>
 <sheets>
@@
 <attribute name="DRAWING_NAME" x="180.34" y="19.05" size="2.54" layer="94"/>
 </instance>
-<instance part="U$1" gate="G$1" x="22.86" y="101.6" smashed="yes" rot="R90">
-<attribute name="NAME" x="20.066" y="111.76" size="1.27" layer="95"/>
-<attribute name="VALUE" x="20.32" y="96.52" size="1.27" layer="96"/>
+<instance part="CONN1" gate="G$1" x="30.48" y="104.14" smashed="yes" rot="R180">
+<attribute name="NAME" x="31.496" y="98.298" size="1.27" layer="95" rot="R180"/>
+<attribute name="VALUE" x="31.496" y="113.792" size="1.27" layer="96" rot="R180"/>
 </instance>
 </instances>
@@
 </segment>
 <segment>
-<wire x1="30.48" y1="106.68" x2="43.18" y2="106.68" width="0.1524" layer="91"/>
-<label x="38.1" y="106.68" size="1.778" layer="95"/>
-<pinref part="U$1" gate="G$1" pin="P3"/>
+<pinref part="CONN1" gate="G$1" pin="P2"/>
+<wire x1="33.02" y1="104.14" x2="45.72" y2="104.14" width="0.1524" layer="91"/>
+<label x="38.1" y="104.14" size="1.778" layer="95"/>
 </segment>
 </net>
@@
 </net>
 <net name="CSN" class="0">
-<segment>
-<wire x1="30.48" y1="109.22" x2="43.18" y2="109.22" width="0.1524" layer="91"/>
-<label x="38.1" y="109.22" size="1.778" layer="95"/>
-<pinref part="U$1" gate="G$1" pin="P4"/>
-</segment>
 <segment>
 <pinref part="IC1" gate="G$1" pin="CSN"/>
@@
 <label x="81.28" y="109.22" size="1.778" layer="95"/>
 </segment>
+<segment>
+<pinref part="CONN1" gate="G$1" pin="P1"/>
+<wire x1="33.02" y1="101.6" x2="45.72" y2="101.6" width="0.1524" layer="91"/>
+<label x="38.1" y="101.6" size="1.778" layer="95"/>
+</segment>
 </net>
 <net name="MISO" class="0">
-<segment>
-<wire x1="30.48" y1="104.14" x2="43.18" y2="104.14" width="0.1524" layer="91"/>
-<label x="38.1" y="104.14" size="1.778" layer="95"/>
-<pinref part="U$1" gate="G$1" pin="P2"/>
-</segment>
 <segment>
 <pinref part="IC1" gate="G$1" pin="MISO"/>
@@
 <label x="81.28" y="104.14" size="1.778" layer="95"/>
 </segment>
+<segment>
+<pinref part="CONN1" gate="G$1" pin="P3"/>
+<wire x1="33.02" y1="106.68" x2="45.72" y2="106.68" width="0.1524" layer="91"/>
+<label x="38.1" y="106.68" size="1.778" layer="95"/>
+</segment>
 </net>
 <net name="MOSI" class="0">
-<segment>
-<wire x1="30.48" y1="101.6" x2="43.18" y2="101.6" width="0.1524" layer="91"/>
-<label x="38.1" y="101.6" size="1.778" layer="95"/>
-<pinref part="U$1" gate="G$1" pin="P1"/>
-</segment>
 <segment>
 <pinref part="IC1" gate="G$1" pin="MOSI"/>
@@
 <label x="81.28" y="101.6" size="1.778" layer="95"/>
 </segment>
-</net>
+<segment>
+<pinref part="CONN1" gate="G$1" pin="P4"/>
+<wire x1="33.02" y1="109.22" x2="45.72" y2="109.22" width="0.1524" layer="91"/>
+<label x="38.1" y="109.22" size="1.778" layer="95"/>
+</segment>
+</net>
