File: 02_pcb/mouse_codename/micromouse2019.sch (EAGLE design)
At the start: 0 parts

Commit message: IRD sheet notes added
Other:
- note added: "The values of R1-R4 will be experimentally determined for optimal illumination and sensitivity."
Changed lines of the file:
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@@
 <layer number="132" name="bAdjust" color="7" fill="1" visible="no" active="yes"/>
 <layer number="144" name="Drill_legend" color="7" fill="1" visible="no" active="yes"/>
-<layer number="150" name="Notes" color="7" fill="1" visible="no" active="yes"/>
+<layer number="150" name="Notes" color="7" fill="1" visible="yes" active="yes"/>
 <layer number="151" name="HeatSink" color="7" fill="1" visible="no" active="yes"/>
 <layer number="152" name="_bDocu" color="7" fill="1" visible="no" active="yes"/>
@@
 <sheet>
 <plain>
+<text x="7.62" y="30.48" size="1.778" layer="150">The values of R1-R4 will be experimentally determined for optimal illumination and sensitivity.</text>
 </plain>
 <instances>
