File: 02_pcb/mouse_codename/micromouse2019.sch (EAGLE design)
At the start: 0 parts

Commit message: pcb route 4th phase
Other:
- note added: "NC_4 and NC_6 connected for soldering stabilization"
- note added: "Note:"
Changed lines of the file:
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@@
 Charge Pump Capacitor (Pin 20) C3 Ceramic, X7R, 2.2nF ±10%, 50V 1
 VLOGIC Bypass Capacitor (Pin 8) C4* Ceramic, X7R, 10nF ±10%, 4V 1</text>
+<text x="147.32" y="134.62" size="1.778" layer="91">Note:</text>
+<text x="149.86" y="132.08" size="1.778" layer="91">NC_4 and NC_6 connected for soldering stabilization</text>
 </plain>
 <instances>
@@
 <wire x1="165.1" y1="104.14" x2="172.72" y2="104.14" width="0.1524" layer="91"/>
 <junction x="172.72" y="104.14"/>
+<pinref part="IC1" gate="G$1" pin="NC_6"/>
+<wire x1="144.78" y1="116.84" x2="172.72" y2="116.84" width="0.1524" layer="91"/>
+<wire x1="172.72" y1="116.84" x2="172.72" y2="109.22" width="0.1524" layer="91"/>
+<junction x="172.72" y="109.22"/>
 </segment>
 <segment>
 <pinref part="IC1" gate="G$1" pin="CLKIN"/>
-<wire x1="111.76" y1="119.38" x2="99.06" y2="119.38" width="0.1524" layer="91"/>
+<wire x1="111.76" y1="119.38" x2="106.68" y2="119.38" width="0.1524" layer="91"/>
+<wire x1="106.68" y1="119.38" x2="99.06" y2="119.38" width="0.1524" layer="91"/>
 <wire x1="99.06" y1="119.38" x2="99.06" y2="116.84" width="0.1524" layer="91"/>
 <pinref part="GND2" gate="1" pin="GND"/>
+<pinref part="IC1" gate="G$1" pin="NC_4"/>
+<wire x1="111.76" y1="109.22" x2="109.22" y2="109.22" width="0.1524" layer="91"/>
+<wire x1="109.22" y1="109.22" x2="106.68" y2="109.22" width="0.1524" layer="91"/>
+<wire x1="106.68" y1="109.22" x2="106.68" y2="119.38" width="0.1524" layer="91"/>
+<junction x="106.68" y="119.38"/>
 </segment>
 <segment>
