File: 02_pcb/mouse_codename/micromouse2019.sch (EAGLE design)
At the start: 2 parts

Commit message: 100k resistor added to SWDIO for bidirectional managment
Other:
- note added: "Note: For SWDIO bidirectional management, the line must be pulled-up on the board (100 KΩ recommended by Arm ® )."
Changed lines of the file:
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@@
 <part name="R9" library="0-micromouse2019" deviceset="R-US_" device="R0402" package3d_urn="urn:adsk.eagle:package:23547/3" value="270R"/>
 <part name="GND9" library="0-micromouse2019" deviceset="GND" device=""/>
+<part name="R10" library="rcl" library_urn="urn:adsk.eagle:library:334" deviceset="R-US_" device="R0402" package3d_urn="urn:adsk.eagle:package:23547/3" value="100k"/>
+<part name="+3V6" library="0-micromouse2019" deviceset="+3V3" device=""/>
 </parts>
 <sheets>
@@
 Note: To reduce leakage it is advisable to configure the I/O as an analog input or to push-pull and
 to set it to “0”.</text>
+<text x="2.54" y="27.94" size="1.778" layer="98">Note:
+For SWDIO bidirectional management, the line must be pulled-up on the board (100 KΩ recommended by Arm ® ).</text>
 </plain>
 <instances>
@@
 <attribute name="VALUE" x="220.98" y="154.94" size="1.778" layer="96"/>
 </instance>
-<instance part="J1" gate="G$1" x="81.28" y="167.64" smashed="yes">
-<attribute name="NAME" x="85.09" y="170.18" size="1.778" layer="95" align="center-left"/>
-<attribute name="VALUE" x="85.09" y="160.02" size="1.778" layer="96" align="center-left"/>
-</instance>
-<instance part="GND6" gate="1" x="78.74" y="157.48" smashed="yes">
-<attribute name="VALUE" x="76.2" y="154.94" size="1.778" layer="96"/>
+<instance part="J1" gate="G$1" x="81.28" y="157.48" smashed="yes">
+<attribute name="NAME" x="85.09" y="160.02" size="1.778" layer="95" align="center-left"/>
+<attribute name="VALUE" x="85.09" y="149.86" size="1.778" layer="96" align="center-left"/>
+</instance>
+<instance part="GND6" gate="1" x="78.74" y="147.32" smashed="yes">
+<attribute name="VALUE" x="76.2" y="144.78" size="1.778" layer="96"/>
 </instance>
 <instance part="RGB1" gate="RGB$" x="127" y="165.1" smashed="yes">
@@
 <instance part="GND9" gate="1" x="215.9" y="71.12" smashed="yes">
 <attribute name="VALUE" x="213.36" y="68.58" size="1.778" layer="96"/>
+</instance>
+<instance part="R10" gate="G$1" x="78.74" y="167.64" smashed="yes" rot="R90">
+<attribute name="NAME" x="77.2414" y="163.83" size="1.778" layer="95" rot="R90"/>
+<attribute name="VALUE" x="82.042" y="163.83" size="1.778" layer="96" rot="R90"/>
+</instance>
+<instance part="+3V6" gate="G$1" x="78.74" y="177.8" smashed="yes">
+<attribute name="VALUE" x="76.2" y="172.72" size="1.778" layer="96" rot="R90"/>
 </instance>
 </instances>
@@
 <wire x1="109.22" y1="165.1" x2="109.22" y2="172.72" width="0.1524" layer="91"/>
 </segment>
+<segment>
+<pinref part="R10" gate="G$1" pin="2"/>
+<wire x1="78.74" y1="172.72" x2="78.74" y2="175.26" width="0.1524" layer="91"/>
+<pinref part="+3V6" gate="G$1" pin="+3V3"/>
+</segment>
 </net>
 <net name="GND" class="0">
@@
 <segment>
 <pinref part="J1" gate="G$1" pin="3"/>
-<wire x1="83.82" y1="162.56" x2="78.74" y2="162.56" width="0.1524" layer="91"/>
-<wire x1="78.74" y1="162.56" x2="78.74" y2="160.02" width="0.1524" layer="91"/>
+<wire x1="83.82" y1="152.4" x2="78.74" y2="152.4" width="0.1524" layer="91"/>
+<wire x1="78.74" y1="152.4" x2="78.74" y2="149.86" width="0.1524" layer="91"/>
 <pinref part="GND6" gate="1" pin="GND"/>
 </segment>
@@
 </segment>
 <segment>
-<wire x1="-12.7" y1="0" x2="2.54" y2="0" width="0.1524" layer="91"/>
-<label x="-10.16" y="0" size="1.778" layer="95"/>
-</segment>
-<segment>
 <wire x1="142.24" y1="101.6" x2="157.48" y2="101.6" width="0.1524" layer="91"/>
 <pinref part="IC1" gate="G$1" pin="PB12"/>
@@
 </segment>
 <segment>
-<wire x1="-12.7" y1="2.54" x2="2.54" y2="2.54" width="0.1524" layer="91"/>
-<label x="-10.16" y="2.54" size="1.778" layer="95"/>
-</segment>
-<segment>
 <wire x1="142.24" y1="99.06" x2="157.48" y2="99.06" width="0.1524" layer="91"/>
 <pinref part="IC1" gate="G$1" pin="PB13"/>
@@
 </segment>
 <segment>
-<wire x1="68.58" y1="167.64" x2="83.82" y2="167.64" width="0.1524" layer="91"/>
-<label x="68.58" y="167.64" size="1.778" layer="95"/>
+<wire x1="68.58" y1="157.48" x2="78.74" y2="157.48" width="0.1524" layer="91"/>
+<label x="68.58" y="157.48" size="1.778" layer="95"/>
 <pinref part="J1" gate="G$1" pin="1"/>
+<wire x1="78.74" y1="157.48" x2="83.82" y2="157.48" width="0.1524" layer="91"/>
+<wire x1="78.74" y1="157.48" x2="78.74" y2="162.56" width="0.1524" layer="91"/>
+<junction x="78.74" y="157.48"/>
+<pinref part="R10" gate="G$1" pin="1"/>
 </segment>
 </net>
@@
 </segment>
 <segment>
-<wire x1="68.58" y1="165.1" x2="83.82" y2="165.1" width="0.1524" layer="91"/>
-<label x="68.58" y="165.1" size="1.778" layer="95"/>
+<wire x1="68.58" y1="154.94" x2="83.82" y2="154.94" width="0.1524" layer="91"/>
+<label x="68.58" y="154.94" size="1.778" layer="95"/>
 <pinref part="J1" gate="G$1" pin="2"/>
 </segment>

Commit message: tNames sized and placed to position
Connections:
- removed net DRAIN_1: CONN1.P1
- removed net DRAIN_2: CONN1.P2
- removed net PTR1: CONN1.P3
- removed net PTR2: CONN1.P4
- removed net VCC: CONN2.P1

Commit message: board updated, strange polygon clearances
Connections:
- net GND: now also CONN1.2; no longer CONN1.1
- net V_BAT_IN: now also CONN1.1; no longer CONN1.2
Changed lines of the file:
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@@
 <attribute name="VALUE" x="137.16" y="116.84" size="1.778" layer="96"/>
 </instance>
-<instance part="CONN1" gate="G$1" x="15.24" y="147.32" smashed="yes" rot="R180">
-<attribute name="NAME" x="17.784359375" y="144.01233125" size="1.78105" layer="95" rot="R180"/>
-<attribute name="VALUE" x="17.784590625" y="154.953759375" size="1.781209375" layer="96" rot="R180"/>
+<instance part="CONN1" gate="G$1" x="20.32" y="149.86" smashed="yes" rot="MR0">
+<attribute name="NAME" x="22.864359375" y="153.16766875" size="1.78105" layer="95" rot="MR0"/>
+<attribute name="VALUE" x="22.864590625" y="142.226240625" size="1.781209375" layer="96" rot="MR0"/>
 </instance>
 </instances>
@@
 </segment>
 <segment>
-<wire x1="20.32" y1="147.32" x2="30.48" y2="147.32" width="0.1524" layer="91"/>
 <wire x1="30.48" y1="147.32" x2="30.48" y2="121.92" width="0.1524" layer="91"/>
 <pinref part="GND8" gate="1" pin="GND"/>
-<pinref part="CONN1" gate="G$1" pin="1"/>
+<pinref part="CONN1" gate="G$1" pin="2"/>
+<wire x1="30.48" y1="147.32" x2="25.4" y2="147.32" width="0.1524" layer="91"/>
 </segment>
 <segment>
@@
 <junction x="96.52" y="149.86"/>
 <junction x="76.2" y="149.86"/>
-<wire x1="20.32" y1="149.86" x2="40.64" y2="149.86" width="0.1524" layer="91"/>
 <wire x1="40.64" y1="149.86" x2="66.04" y2="149.86" width="0.1524" layer="91"/>
 <wire x1="66.04" y1="149.86" x2="76.2" y2="149.86" width="0.1524" layer="91"/>
@@
 <pinref part="R1" gate="G$1" pin="2"/>
 <wire x1="40.64" y1="147.32" x2="40.64" y2="149.86" width="0.1524" layer="91"/>
-<junction x="40.64" y="149.86"/>
 <wire x1="96.52" y1="93.98" x2="96.52" y2="96.52" width="0.1524" layer="91"/>
 <junction x="96.52" y="96.52"/>
 <label x="48.26" y="149.86" size="1.778" layer="95"/>
-<pinref part="CONN1" gate="G$1" pin="2"/>
+<pinref part="CONN1" gate="G$1" pin="1"/>
+<wire x1="25.4" y1="149.86" x2="40.64" y2="149.86" width="0.1524" layer="91"/>
+<junction x="40.64" y="149.86"/>
 </segment>
 </net>

Commit message: I2C pull up resistors added
Parts:
- added R1, R2: 4k7, 0-micromouse2019:R-US_R0402
Connections:
- new net +3V3: R1.2, R2.2
- new net AD0: R1.2
- new net BOOT1: R2.2
- new net BTN_BOOT0: R1.1
- new net IRD1: R1.2
- new net IRD2: R2.2
- new net SCL: R1.1
- new net SDA: R2.1
- new net V_BAT_LEVEL: R1.1, R2.2
- net GND: now also R1.1, R2.1
- net V_BAT_IN: now also R1.2
Changed lines of the file:
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@@
 <part name="CONN1" library="0-micromouse2019" deviceset="CONN_IRD_VCC" device="" package3d_urn="urn:adsk.eagle:package:9165697/2"/>
 <part name="CONN2" library="0-micromouse2019" deviceset="CONN_IRD_VCC" device="" package3d_urn="urn:adsk.eagle:package:9165697/2"/>
+<part name="R1" library="0-micromouse2019" deviceset="R-US_" device="R0402" package3d_urn="urn:adsk.eagle:package:23547/3" value="4k7"/>
+<part name="+3V6" library="0-micromouse2019" deviceset="+3V3" device=""/>
+<part name="+3V7" library="0-micromouse2019" deviceset="+3V3" device=""/>
+<part name="R2" library="0-micromouse2019" deviceset="R-US_" device="R0402" package3d_urn="urn:adsk.eagle:package:23547/3" value="4k7"/>
 </parts>
 <sheets>
@@
 <attribute name="NAME" x="66.04" y="147.32" size="2.032" layer="95" align="bottom-center"/>
 </moduleinst>
-<moduleinst name="IMU" module="INERTIAL_MEASUREMENT_UNIT" x="66.04" y="71.12">
-<attribute name="NAME" x="66.04" y="71.12" size="2.032" layer="95" align="bottom-center"/>
+<moduleinst name="IMU" module="INERTIAL_MEASUREMENT_UNIT" x="50.8" y="71.12">
+<attribute name="NAME" x="50.8" y="71.12" size="2.032" layer="95" align="bottom-center"/>
 </moduleinst>
 <moduleinst name="MOT" module="MOTOR_DRIVER" x="187.96" y="104.14">
 <attribute name="NAME" x="187.96" y="104.14" size="2.032" layer="95" align="bottom-center"/>
 </moduleinst>
-<moduleinst name="EPR" module="ENCODER_PORT" x="66.04" y="88.9">
-<attribute name="NAME" value="EPR" x="68.58" y="83.82" size="2.032" layer="95" align="bottom-center"/>
+<moduleinst name="EPR" module="ENCODER_PORT" x="50.8" y="88.9">
+<attribute name="NAME" value="EPR" x="53.34" y="83.82" size="2.032" layer="95" align="bottom-center"/>
 </moduleinst>
 <moduleinst name="BTP" module="WIRELESS_MODUL_PORT" x="124.46" y="30.48">
 <attribute name="NAME" value="BTP" x="124.46" y="25.4" size="2.032" layer="95" align="bottom-center"/>
 </moduleinst>
-<moduleinst name="EPL" module="ENCODER_PORT" x="66.04" y="104.14">
-<attribute name="NAME" value="EPL" x="68.58" y="99.06" size="2.032" layer="95" align="bottom-center"/>
+<moduleinst name="EPL" module="ENCODER_PORT" x="50.8" y="104.14">
+<attribute name="NAME" value="EPL" x="53.34" y="99.06" size="2.032" layer="95" align="bottom-center"/>
 </moduleinst>
 <moduleinst name="MCU" module="MICROCONTROLLER" x="129.54" y="86.36">
@@
 <attribute name="VALUE" x="119.38" y="124.46" size="1.778" layer="96" rot="R90"/>
 </instance>
-<instance part="+3V3" gate="G$1" x="35.56" y="116.84" smashed="yes">
-<attribute name="VALUE" x="33.02" y="111.76" size="1.778" layer="96" rot="R90"/>
-</instance>
-<instance part="GND2" gate="1" x="40.64" y="55.88" smashed="yes">
-<attribute name="VALUE" x="38.1" y="53.34" size="1.778" layer="96"/>
+<instance part="+3V3" gate="G$1" x="20.32" y="116.84" smashed="yes">
+<attribute name="VALUE" x="17.78" y="111.76" size="1.778" layer="96" rot="R90"/>
+</instance>
+<instance part="GND2" gate="1" x="25.4" y="55.88" smashed="yes">
+<attribute name="VALUE" x="22.86" y="53.34" size="1.778" layer="96"/>
 </instance>
 <instance part="GND3" gate="1" x="142.24" y="45.72" smashed="yes">
@@
 <attribute name="NAME" x="99.06" y="127.254" size="1.27" layer="95"/>
 <attribute name="VALUE" x="99.06" y="125.222" size="1.27" layer="96"/>
+</instance>
+<instance part="R1" gate="G$1" x="80.264" y="78.74" smashed="yes" rot="R90">
+<attribute name="NAME" x="78.5114" y="75.946" size="1.778" layer="95" rot="R90"/>
+<attribute name="VALUE" x="83.566" y="74.93" size="1.778" layer="96" rot="R90"/>
+</instance>
+<instance part="+3V6" gate="G$1" x="91.44" y="86.36" smashed="yes">
+<attribute name="VALUE" x="89.662" y="81.534" size="1.778" layer="96" rot="R90"/>
+</instance>
+<instance part="+3V7" gate="G$1" x="80.264" y="86.36" smashed="yes">
+<attribute name="VALUE" x="78.74" y="81.534" size="1.778" layer="96" rot="R90"/>
+</instance>
+<instance part="R2" gate="G$1" x="91.44" y="77.724" smashed="yes" rot="R90">
+<attribute name="NAME" x="89.6874" y="75.438" size="1.778" layer="95" rot="R90"/>
+<attribute name="VALUE" x="94.742" y="75.184" size="1.778" layer="96" rot="R90"/>
 </instance>
 </instances>
@@
 </segment>
 <segment>
-<wire x1="40.64" y1="99.06" x2="40.64" y2="83.82" width="0.1524" layer="91"/>
+<wire x1="25.4" y1="99.06" x2="25.4" y2="83.82" width="0.1524" layer="91"/>
 <portref moduleinst="IMU" port="GND"/>
-<wire x1="40.64" y1="83.82" x2="40.64" y2="66.04" width="0.1524" layer="91"/>
-<wire x1="40.64" y1="66.04" x2="43.18" y2="66.04" width="0.1524" layer="91"/>
-<wire x1="40.64" y1="66.04" x2="40.64" y2="58.42" width="0.1524" layer="91"/>
-<junction x="40.64" y="66.04"/>
+<wire x1="25.4" y1="83.82" x2="25.4" y2="66.04" width="0.1524" layer="91"/>
+<wire x1="25.4" y1="66.04" x2="27.94" y2="66.04" width="0.1524" layer="91"/>
+<wire x1="25.4" y1="66.04" x2="25.4" y2="58.42" width="0.1524" layer="91"/>
+<junction x="25.4" y="66.04"/>
 <pinref part="GND2" gate="1" pin="GND"/>
 <portref moduleinst="EPL" port="GND"/>
-<wire x1="43.18" y1="99.06" x2="40.64" y2="99.06" width="0.1524" layer="91"/>
+<wire x1="27.94" y1="99.06" x2="25.4" y2="99.06" width="0.1524" layer="91"/>
 <portref moduleinst="EPR" port="GND"/>
-<wire x1="43.18" y1="83.82" x2="40.64" y2="83.82" width="0.1524" layer="91"/>
-<junction x="40.64" y="83.82"/>
+<wire x1="27.94" y1="83.82" x2="25.4" y2="83.82" width="0.1524" layer="91"/>
+<junction x="25.4" y="83.82"/>
 </segment>
 <segment>
@@
 </segment>
 <segment>
-<wire x1="35.56" y1="93.98" x2="35.56" y2="109.22" width="0.1524" layer="91"/>
+<wire x1="20.32" y1="93.98" x2="20.32" y2="109.22" width="0.1524" layer="91"/>
 <portref moduleinst="IMU" port="+3V3"/>
-<wire x1="43.18" y1="76.2" x2="35.56" y2="76.2" width="0.1524" layer="91"/>
-<wire x1="35.56" y1="76.2" x2="35.56" y2="93.98" width="0.1524" layer="91"/>
-<wire x1="35.56" y1="109.22" x2="35.56" y2="114.3" width="0.1524" layer="91"/>
+<wire x1="27.94" y1="76.2" x2="20.32" y2="76.2" width="0.1524" layer="91"/>
+<wire x1="20.32" y1="76.2" x2="20.32" y2="93.98" width="0.1524" layer="91"/>
+<wire x1="20.32" y1="109.22" x2="20.32" y2="114.3" width="0.1524" layer="91"/>
 <pinref part="+3V3" gate="G$1" pin="+3V3"/>
 <portref moduleinst="EPL" port="+3V3"/>
-<wire x1="43.18" y1="109.22" x2="35.56" y2="109.22" width="0.1524" layer="91"/>
-<junction x="35.56" y="109.22"/>
+<wire x1="27.94" y1="109.22" x2="20.32" y2="109.22" width="0.1524" layer="91"/>
+<junction x="20.32" y="109.22"/>
 <portref moduleinst="EPR" port="+3V3"/>
-<wire x1="43.18" y1="93.98" x2="35.56" y2="93.98" width="0.1524" layer="91"/>
-<junction x="35.56" y="93.98"/>
+<wire x1="27.94" y1="93.98" x2="20.32" y2="93.98" width="0.1524" layer="91"/>
+<junction x="20.32" y="93.98"/>
 </segment>
 <segment>
@@
 <wire x1="220.98" y1="106.68" x2="220.98" y2="121.92" width="0.1524" layer="91"/>
 <pinref part="+3V5" gate="G$1" pin="+3V3"/>
+</segment>
+<segment>
+<pinref part="+3V7" gate="G$1" pin="+3V3"/>
+<pinref part="R1" gate="G$1" pin="2"/>
+</segment>
+<segment>
+<pinref part="R2" gate="G$1" pin="2"/>
+<pinref part="+3V6" gate="G$1" pin="+3V3"/>
+<wire x1="91.44" y1="82.804" x2="91.44" y2="83.82" width="0.1524" layer="91"/>
 </segment>
 </net>
@@
 <portref moduleinst="IMU" port="SCL"/>
 <portref moduleinst="MCU" port="IMU1_SCL"/>
-<wire x1="88.9" y1="73.66" x2="96.52" y2="73.66" width="0.1524" layer="91"/>
+<wire x1="73.66" y1="73.66" x2="80.264" y2="73.66" width="0.1524" layer="91"/>
+<pinref part="R1" gate="G$1" pin="1"/>
+<wire x1="80.264" y1="73.66" x2="96.52" y2="73.66" width="0.1524" layer="91"/>
+<junction x="80.264" y="73.66"/>
 </segment>
 </net>
@@
 <portref moduleinst="IMU" port="SDA"/>
 <portref moduleinst="MCU" port="IMU1_SDA"/>
-<wire x1="88.9" y1="68.58" x2="96.52" y2="68.58" width="0.1524" layer="91"/>
+<wire x1="73.66" y1="68.58" x2="91.44" y2="68.58" width="0.1524" layer="91"/>
+<wire x1="91.44" y1="68.58" x2="96.52" y2="68.58" width="0.1524" layer="91"/>
+<pinref part="R2" gate="G$1" pin="1"/>
+<wire x1="91.44" y1="72.644" x2="91.44" y2="68.58" width="0.1524" layer="91"/>
+<junction x="91.44" y="68.58"/>
 </segment>
 </net>
@@
 <portref moduleinst="EPL" port="ENC_CHA"/>
 <portref moduleinst="MCU" port="ENC_LEFT_CHA"/>
-<wire x1="88.9" y1="106.68" x2="96.52" y2="106.68" width="0.1524" layer="91"/>
+<wire x1="73.66" y1="106.68" x2="96.52" y2="106.68" width="0.1524" layer="91"/>
 </segment>
 </net>
@@
 <portref moduleinst="EPL" port="ENC_CHB"/>
 <portref moduleinst="MCU" port="ENC_LEFT_CHB"/>
-<wire x1="88.9" y1="104.14" x2="96.52" y2="104.14" width="0.1524" layer="91"/>
+<wire x1="73.66" y1="104.14" x2="96.52" y2="104.14" width="0.1524" layer="91"/>
 </segment>
 </net>
@@
 <portref moduleinst="EPR" port="ENC_CHA"/>
 <portref moduleinst="MCU" port="ENC_RIGHT_CHA"/>
-<wire x1="88.9" y1="91.44" x2="96.52" y2="91.44" width="0.1524" layer="91"/>
+<wire x1="73.66" y1="91.44" x2="96.52" y2="91.44" width="0.1524" layer="91"/>
 </segment>
 </net>
@@
 <portref moduleinst="EPR" port="ENC_CHB"/>
 <portref moduleinst="MCU" port="ENC_RIGHT_CHB"/>
-<wire x1="88.9" y1="88.9" x2="96.52" y2="88.9" width="0.1524" layer="91"/>
-</segment>
-</net>
+<wire x1="73.66" y1="88.9" x2="96.52" y2="88.9" width="0.1524" layer="91"/>
+</segment>
+</net>
